File: flip-flop-NE555-timer.kicad_pcb (KiCad board)
At the start: 2 copper layers, 25 x 27 mm, 10 parts, among them J2 Conn_01x02_Pin, U1 NE555P

Commit message: Add files via upload
Parts:
- moved U1 16.6 mm to (127.2, 70.2)
- moved C2 16.6 mm to (132.0, 85.0)
- moved C3 16.6 mm to (123.0, 72.5)
- moved D1 16.6 mm to (139.5, 66.0)
- moved D2 16.6 mm to (142.0, 84.0)
- moved J2 16.6 mm to (123.0, 84.0)
- moved R1 16.6 mm to (143.3, 72.0)
- moved R2 16.6 mm to (138.2, 77.0)
- moved R3 16.6 mm to (131.0, 65.0)
- moved R4 16.6 mm to (123.5, 65.0)
